Commit message: lanch better

File: server_ws/src/nav_bot1/description/xiao_geek_robot.xacro (robot description, xacro)
@@ -39,5 +39,5 @@
     <parent link="base_link"/>
     <child link="left_track"/>
-    <origin xyz="0 0.105 0.05" rpy="0 0 ${pi/2}"/>
+    <origin xyz="0 0.175 0" rpy="-${pi/2} 0 0"/>
     <axis xyz="0 0 1"/>
   </joint>
@@ -45,5 +45,5 @@
     <visual>
       <geometry>
-        <cylinder radius="0.03" length="0.02"/>
+        <cylinder radius="0.05" length="0.02"/>
       </geometry>
       <material name="blue"/>
@@ -51,5 +51,5 @@
     <collision>
       <geometry>
-        <cylinder radius="0.03" length="0.02"/>
+        <cylinder radius="0.05" length="0.02"/>
       </geometry>
     </collision>
@@ -62,5 +62,5 @@
     <parent link="base_link"/>
     <child link="right_track"/>
-    <origin xyz="0 -0.105 0.05" rpy="0 0 ${pi/2}"/>
+    <origin xyz="0 -0.175 0" rpy="${pi/2} 0 0"/>
     <axis xyz="0 0 -1"/>
   </joint>
@@ -120,20 +120,3 @@
     </xacro:inertial_box>
   </link>
-  <!-- 3.5 inch Touch Display -->
-  <joint name="touchscreen_joint" type="fixed">
-    <parent link="chassis"/>
-    <child link="touchscreen"/>
-    <origin xyz="-0.05 0 0.09"/>
-  </joint>
-  <link name="touchscreen">
-    <visual>
-      <geometry>
-        <box size="0.09 0.05 0.007"/>
-      </geometry>
-      <material name="white"/>
-    </visual>
-    <xacro:inertial_box mass="0.08" x="0.09" y="0.05" z="0.007">
-      <origin xyz="0 0 0"/>
-    </xacro:inertial_box>
-  </link>
 </robot>

File: server_ws/src/nav_bot1/description/xiaor_geek_robot.urdf.xacro (robot description, xacro)
@@ -1,5 +1,5 @@
 <?xml version="1.0"?>
 <robot xmlns:xacro="http://www.ros.org/wiki/xacro" name="xiaor_geek_robot">
-  <xacro:include filename="intertial_macros.xacro"/>
+  <xacro:include filename="inertial_macros.xacro"/>
   <xacro:include filename="xiao_geek_robot.xacro"/>
 </robot>

Commit message: urdf 2nd try

File: server_ws/src/nav_bot1/description/xiao_geek_robot.xacro (robot description, xacro)
@@ -35,50 +35,54 @@
     </xacro:inertial_box>
   </link>
-  <!-- Left track wheel -->
-  <joint name="left_track_joint" type="continuous">
-    <parent link="base_link"/>
-    <child link="left_track"/>
-    <origin xyz="0 0.175 0" rpy="-${pi/2} 0 0"/>
-    <axis xyz="0 0 1"/>
-  </joint>
-  <link name="left_track">
-    <visual>
-      <geometry>
-        <cylinder radius="0.05" length="0.02"/>
-      </geometry>
-      <material name="blue"/>
-    </visual>
-    <collision>
-      <geometry>
-        <cylinder radius="0.05" length="0.02"/>
-      </geometry>
-    </collision>
-    <xacro:inertial_cylinder mass="0.2" length="0.02" radius="0.03">
-      <origin xyz="0 0 0"/>
-    </xacro:inertial_cylinder>
-  </link>
-  <!-- Right track wheel -->
-  <joint name="right_track_joint" type="continuous">
-    <parent link="base_link"/>
-    <child link="right_track"/>
-    <origin xyz="0 -0.175 0" rpy="${pi/2} 0 0"/>
-    <axis xyz="0 0 -1"/>
-  </joint>
-  <link name="right_track">
-    <visual>
-      <geometry>
-        <cylinder radius="0.03" length="0.02"/>
-      </geometry>
-      <material name="blue"/>
-    </visual>
-    <collision>
-      <geometry>
-        <cylinder radius="0.03" length="0.02"/>
-      </geometry>
-    </collision>
-    <xacro:inertial_cylinder mass="0.2" length="0.02" radius="0.03">
-      <origin xyz="0 0 0"/>
-    </xacro:inertial_cylinder>
-  </link>
+    <!-- LEFT WHEEL -->
+    <joint name="left_wheel_joint" type="continuous">
+        <parent link="base_link"/>
+        <child link="left_wheel"/>
+        <origin xyz="0.0 0.09 0.035" rpy="0 0 0"/>
+        <axis xyz="0 1 0"/>
+    </joint>
+    <link name="left_wheel">
+        <visual>
+            <origin xyz="0 0 0" rpy="0 0 0"/>
+            <geometry>
+                <cylinder radius="0.045" length="0.02"/>
+            </geometry>
+            <material name="black"/>
+        </visual>
+        <collision>
+            <origin xyz="0 0 0" rpy="0 0 0"/>
+            <geometry>
+                <cylinder radius="0.045" length="0.02"/>
+            </geometry>
+        </collision>
+        <xacro:inertial_cylinder mass="0.15" length="0.02" radius="0.045">
+            <origin xyz="0 0 0" rpy="0 0 0"/>
+        </xacro:inertial_cylinder>
+    </link>
+    <!-- RIGHT WHEEL -->
+    <joint name="right_wheel_joint" type="continuous">
+        <parent link="base_link"/>
+        <child link="right_wheel"/>
+        <origin xyz="0.0 -0.09 0.035" rpy="0 0 0"/>
+        <axis xyz="0 1 0"/>
+    </joint>
+    <link name="right_wheel">
+        <visual>
+            <origin xyz="0 0 0" rpy="0 0 0"/>
+            <geometry>
+                <cylinder radius="0.045" length="0.02"/>
+            </geometry>
+            <material name="black"/>
+        </visual>
+        <collision>
+            <origin xyz="0 0 0" rpy="0 0 0"/>
+            <geometry>
+                <cylinder radius="0.045" length="0.02"/>
+            </geometry>
+        </collision>
+        <xacro:inertial_cylinder mass="0.15" length="0.02" radius="0.045">
+            <origin xyz="0 0 0" rpy="0 0 0"/>
+        </xacro:inertial_cylinder>
+    </link>
   <!-- RPLidar -->
   <joint name="lidar_joint" type="fixed">

Commit message: updates

File: server_ws/src/nav_bot1/description/xiao_geek_robot.xacro (robot description, xacro)
@@ -93,5 +93,5 @@
     <parent link="chassis"/>
     <child link="lidar"/>
-    <origin xyz="0.07 0 0.1"/>
+    <origin xyz="0.25 0 0.15"/>
   </joint>
   <link name="lidar">
@@ -108,5 +108,5 @@
     </collision>
     <xacro:inertial_cylinder mass="0.15" length="0.03" radius="0.035">
-      <origin xyz="0 0 0"/>
+      <origin xyz="0.25 0 0.15"/>
     </xacro:inertial_cylinder>
   </link>
@@ -115,5 +115,5 @@
     <parent link="chassis"/>
     <child link="camera"/>
-    <origin xyz="0.05 0 0.1"/>
+    <origin xyz="0.15 0 0.15"/>
   </joint>
   <link name="camera">
@@ -125,5 +125,5 @@
     </visual>
     <xacro:inertial_box mass="0.05" x="0.025" y="0.025" z="0.02">
-      <origin xyz="0 0 0"/>
+      <origin xyz="0.15 0 0.15"/>
     </xacro:inertial_box>
   </link>

Commit message: colors

File: server_ws/src/nav_bot1/description/xiao_geek_robot.xacro (robot description, xacro)
@@ -4,16 +4,10 @@
   <xacro:include filename="inertial_macros.xacro"/>
   <!-- Materials -->
-    <material name="white">
-        <color rgba="1 1 1 1" />
-    </material>
-    <material name="orange">
-        <color rgba="1 0.3 0.1 1"/>
-    </material>
-    <material name="blue">
-        <color rgba="0.2 0.2 1 1"/>
-    </material>
-    <material name="black">
-        <color rgba="0 0 0 1"/>
-    </material>
+    <material name="black"><color rgba="0 0 0 1"/></material>
+    <material name="white"><color rgba="1 1 1 1"/></material>
+    <material name="silver"><color rgba="0.75 0.75 0.75 1"/></material>
+    <material name="blue"><color rgba="0.2 0.2 1 1"/></material>
+    <material name="green"><color rgba="0.2 1 0.2 1"/></material>
+    <material name="red"><color rgba="1 0.1 0.1 1"/></material>
     <!-- BASE LINK -->
     <link name="base_link">

Commit message: caster wheel

File: server_ws/src/nav_bot1/description/xiao_geek_robot.xacro (robot description, xacro)
@@ -122,3 +122,20 @@
     </xacro:inertial_box>
   </link>
+  <!-- CASTER WHEEL NO PURPOSE ONLY FOR SIMULATION AND GEOMETRY/PHYSICS -->
+    <link name="caster_wheel">
+        <visual>
+            <geometry>
+                <sphere radius="0.05"/>
+            </geometry>
+            <material name="black"/>
+        </visual>
+        <collision>
+            <geometry>
+                <sphere radius="0.05"/>
+            </geometry>
+        </collision>
+        <xacro:inertial_sphere mass="0.1" radius="0.05">
+            <origin xyz="0 0 0" rpy="0 0 0"/>
+        </xacro:inertial_sphere>
+    </link>
 </robot>

Commit message: working urdf

File: server_ws/src/nav_bot1/description/xiao_geek_robot.xacro (robot description, xacro)
@@ -109,5 +109,5 @@
     <parent link="chassis"/>
     <child link="camera"/>
-    <origin xyz="0.15 0 0.15"/>
+    <origin xyz="0.15 0 0.25"/>
   </joint>
   <link name="camera">
@@ -119,23 +119,28 @@
     </visual>
     <xacro:inertial_box mass="0.05" x="0.025" y="0.025" z="0.02">
-      <origin xyz="0.15 0 0.15"/>
+      <origin xyz="0.15 0 0.25"/>
     </xacro:inertial_box>
   </link>
   <!-- CASTER WHEEL NO PURPOSE ONLY FOR SIMULATION AND GEOMETRY/PHYSICS -->
-    <link name="caster_wheel">
-        <visual>
-            <geometry>
-                <sphere radius="0.05"/>
-            </geometry>
-            <material name="black"/>
-        </visual>
-        <collision>
-            <geometry>
-                <sphere radius="0.05"/>
-            </geometry>
-        </collision>
-        <xacro:inertial_sphere mass="0.1" radius="0.05">
-            <origin xyz="0 0 0" rpy="0 0 0"/>
-        </xacro:inertial_sphere>
-    </link>
+  <joint name="caster_wheel_joint" type="fixed">
+    <parent link="chassis"/>
+    <child link="caster_wheel"/>
+    <origin xyz="0.24 0 0"/>
+  </joint>
+  <link name="caster_wheel">
+      <visual>
+          <geometry>
+              <sphere radius="0.05"/>
+          </geometry>
+          <material name="black"/>
+      </visual>
+      <collision>
+          <geometry>
+              <sphere radius="0.05"/>
+          </geometry>
+      </collision>
+      <xacro:inertial_sphere mass="0.1" radius="0.05">
+          <origin xyz="0 0 0" rpy="0 0 0"/>
+      </xacro:inertial_sphere>
+  </link>
 </robot>
